File: MainBoard.Pic18F4550.Option2/MainBoard.sch (KiCad schematic (older format))
At the start: 91 parts, among them CON1 POWER_BUS, CON2 ICSP_CON, CON3 USB_CON, J1 RESET_CON, J2 SATA_PLUG _22P_SMT, J4 SATA_PLUG _22P_SMT, P1 DEBUG_HEADER_21P, P2 DEBUG_HEADER_21P, Q1 2N2222-SOT23, U1 PIC18F4550-I/P, U3 PCF85263A, Y1 Crystal, Y2 32.768KHZ

Commit message: Revision de PCBs + generacion nuevos gerber
  - Se hacen ligeras correcciones en los PCBs (5)
  - Se genera nuevamente archivo PCBs combinados
  - Se generan nuevos archivos gerber
Changed lines of the file:
@@
 LIBS:74xx
 LIBS:cmos4000
-LIBS:PIC18F4550-I_P
 LIBS:MainBoard-cache
 EELAYER 25 0
@@
 Entry Wire Line
 	3900 2650 4000 2750
-Entry Wire Line
-	3900 2750 4000 2850
 Entry Wire Line
 	3900 2850 4000 2950
@@
 RB7
 Wire Wire Line
-	4200 2850 4000 2850
-Wire Wire Line
 	4000 2950 4200 2950
 Wire Wire Line
@@
 Text Label 1650 1600 0    39   ~ 0
 PC1
+$Comp
+L GNDD #PWR?
+U 1 1 5A767BCA
+P 4250 3350
+F 0 "#PWR?" H 4250 3100 50  0001 C CNN
+F 1 "GNDD" V 4350 3350 50  0000 C CNN
+F 2 "" H 4250 3350 50  0001 C CNN
+F 3 "" H 4250 3350 50  0001 C CNN
+	1    4250 3350
+	0    1    1    0
+$EndComp
+$Comp
+L GNDD #PWR?
+U 1 1 5A76867F
+P 4100 2850
+F 0 "#PWR?" H 4100 2600 50  0001 C CNN
+F 1 "GNDD" V 4100 2800 50  0000 C CNN
+F 2 "" H 4100 2850 50  0001 C CNN
+F 3 "" H 4100 2850 50  0001 C CNN
+	1    4100 2850
+	0    1    1    0
+$EndComp
+Wire Wire Line
+	4200 2850 4100 2850
 $EndSCHEMATC
