File: MergedPcbs/KicadFiles/MergedPcbs.kicad_pcb (KiCad board)
At the start: 2 copper layers, 324 parts, among them CON1 POWER_BUS, CON1 USB_CON, CON2 ICSP_CON, CON3 USB_CON, J1 DEBUG_CON_01X08, J1 DEBUG_CON_01X09, J1 RESET_CON, J1 RESET_CON_01X02, J1 VIKING_CON_9P, J10 IO_CON_8P, J11 PORTB_CON_6P, J12 PORTCD_CON_5P, J13 PORTAE_CON_8P, J2 GPIB_CON_9P, J2 POWER_CON_01X02, J2 SATA_PLUG _22P_SMT, J2 VIKING_CON_01X09, J3 GPIB_CON_9P, J3 VIKING_CON_01X09, J3 VIKING_CON_9P, J4 GPIB_CON_9P, J4 SATA_CON_14P, J4 SATA_PLUG _22P_SMT, J4 SATA_PLUG_CON_14P, J5 POWER_CON_01X06, J6 VIKING_CON_01X09, J7 VIKING_CON_01X09, J8 RESET_CON_01X02, J9 IO_CON_8P, P1 DEBUG_HEADER_21P, P1 PORTB_CON_9P, P1 PWR_IN_2P, P2 DEBUG_HEADER_21P, P2 PORTA_CON_6P, P2 PWR_OUT_4P, P3 PORTE_CON_3P, P4 SATA_CON_L_13P, P5 PORTCD_H_CON_7P, P6 PORTCD_L_CON_8P, P7 SATA_CON_R_13P, Q1 2N2222-SOT23, Q1 2N3904, U1 MC33996EKR2, U1 PCA6416A, U1 PIC18F4550-I/P, U1 SP34063A, U2 PIC18F4550-I/P, U2 SPX29152, U3 MC33996EKR2, U3 PCF85263A, U4 MC33996EKR2, U5 PCA6416A, Y1 20MHZ, Y1 Crystal, Y2 32.768KHZ

Commit message: Revision de PCbs + generacion de nuevos archivos Gerber
  - Se corrigen pads de pin headers
  - Se revisan
  - MainBoard option 2
  - PortExpander MC33996.Option3
  - GpibPortExpanderPCA6408A.Option3
  - Se generan Gerber + Vistas 3D
Parts:
- removed the C1 at (258.4, 71.4)
- removed the C1 at (233.6, 44.3)
- removed the C1 at (26.7, 136.1)
- removed the C1 at (237.4, 148.5)
- removed the C1 at (138.0, 58.7)
- removed the C1 at (94.3, 152.8)
- removed the C10 at (127.4, 144.4)
- removed the C11 at (127.4, 150.5)
- removed the C12 at (120.8, 118.4)
- removed the C13 at (190.1, 118.4)
- removed the C2 at (266.4, 71.4)
- removed the C2 at (229.9, 39.5)
- removed the C2 at (25.4, 143.1)
- removed the C2 at (236.1, 155.4)
- removed the C2 at (138.0, 64.8)
- removed the C2 at (95.1, 183.0)
- removed the C3 at (47.0, 124.1)
- removed the C3 at (257.7, 136.4)
- removed the C3 at (137.7, 25.7)
- removed the C3 at (164.1, 137.6)
- removed the C4 at (54.6, 125.3)
- removed the C4 at (265.3, 137.7)
- removed the C4 at (147.7, 73.8)
- removed the C4 at (182.3, 145.2)
- removed the C5 at (57.1, 143.1)
- removed the C5 at (267.8, 155.4)
- removed the C5 at (140.0, 52.8)
- removed the C5 at (91.2, 147.5)
- removed the C6 at (59.1, 150.1)
- removed the C6 at (269.7, 162.4)
- removed the C6 at (178.1, 49.8)
- removed the C6 at (92.0, 177.6)
- removed the C7 at (31.1, 153.3)
- removed the C7 at (241.8, 165.6)
- removed the C7 at (190.4, 145.2)
- removed the C8 at (33.7, 160.3)
- removed the C8 at (244.3, 172.6)
- removed the C9 at (59.1, 154.6)
- removed the C9 at (269.7, 166.9)
- removed the C9 at (136.2, 160.4)
- removed the CON1 at (190.2, 78.1)
- removed the CON1 at (153.1, 178.7)
- removed the D1 at (254.1, 91.6)
- removed the D1 at (33.0, 142.5)
- removed the D1 at (243.7, 154.8)
- removed the D1 at (183.5, 63.5)
- removed the D1 at (174.3, 165.5)
- removed the D10 at (259.7, 104.7)
- removed the D10 at (179.9, 178.5)
- removed the D11 at (257.2, 104.7)
- removed the D11 at (177.5, 178.5)
- removed the D12 at (254.3, 104.7)
- removed the D12 at (174.6, 178.5)
- removed the D13 at (272.6, 104.7)
- removed the D13 at (192.9, 178.5)
- removed the D14 at (269.9, 104.7)
- removed the D14 at (190.2, 178.5)
- removed the D15 at (267.1, 104.7)
- removed the D15 at (187.4, 178.5)
- removed the D16 at (264.7, 104.7)
- removed the D16 at (185.0, 178.5)
- removed D17, D18: LED, LEDs:LED_0805_HandSoldering
- removed D19, D20: SP1003, CenditFootprints:SP1003-01ETG
- removed the D2 at (256.7, 91.5)
- removed the D2 at (28.1, 124.7)
- removed the D2 at (238.8, 137.0)
- removed the D2 at (180.5, 63.5)
- removed the D2 at (177.0, 165.3)
- removed the D3 at (259.3, 91.5)
- removed the D3 at (62.9, 120.3)
- removed the D3 at (273.6, 132.6)
- removed the D3 at (186.3, 70.9)
- removed the D3 at (179.5, 165.3)
- removed the D4 at (262.1, 91.5)
- removed the D4 at (182.3, 165.3)
- removed the D5 at (264.7, 91.5)
- removed the D5 at (185.0, 165.3)
- removed the D6 at (267.4, 91.5)
- removed the D6 at (187.7, 165.3)
- removed the D7 at (269.9, 91.5)
- removed the D7 at (190.2, 165.3)
- removed the D8 at (272.6, 91.5)
- removed the D8 at (192.9, 165.3)
- removed the D9 at (262.2, 104.7)
- removed the D9 at (182.5, 178.5)
- removed the J1 at (238.4, 79.2)
- removed the J1 at (267.5, 27.7)
- removed the J1 at (141.9, 26.9)
- removed the J1 at (118.5, 167.7)
- removed J10, J9: IO_CON_8P, Pin_Headers:Pin_Header_Straight_1x09_Pitch2.54mm
- removed J11: PORTB_CON_6P, Pin_Headers:Pin_Header_Straight_1x06_Pitch2.54mm
- removed J12: PORTCD_CON_5P, Pin_Headers:Pin_Header_Straight_1x05_Pitch2.54mm
- removed J13: PORTAE_CON_8P, Pin_Headers:Pin_Header_Straight_1x08_Pitch2.54mm
- removed the J2 at (271.3, 96.4)
- removed the J2 at (256.9, 29.3)
- removed the J2 at (192.7, 55.6)
- removed the J2 at (191.5, 170.1)
- removed the J3 at (271.3, 99.8)
- removed the J3 at (256.9, 26.0)
- removed the J3 at (118.5, 164.4)
- removed the J4 at (275.2, 36.1)
- removed the J4 at (191.5, 173.5)
- removed J5: POWER_CON_01X06, Pin_Headers:Pin_Header_Straight_1x06_Pitch2.54mm
- removed J6, J7: VIKING_CON_01X09, Pin_Headers:Pin_Header_Straight_1x09_Pitch2.54mm
- removed J8: RESET_CON_01X02, Pin_Headers:Pin_Header_Straight_1x02_Pitch2.54mm
- removed the JP1 at (188.8, 60.7)
- removed the JP1 at (203.6, 152.1)
- removed the JP2 at (200.0, 152.1)
- removed the L1 at (45.7, 138.0)
- removed the L1 at (256.4, 150.4)
- removed the L2 at (58.4, 133.6)
- removed the L2 at (269.1, 145.9)
- removed the LS1 at (97.6, 125.8)
- removed the P1 at (24.8, 126.0)
- removed the P1 at (235.5, 138.3)
- removed the P1 at (185.4, 49.3)
- removed the P2 at (25.4, 153.3)
- removed the P2 at (236.1, 165.6)
- removed the P2 at (139.2, 31.5)
- removed P3: PORTE_CON_3P, Pin_Headers:Pin_Header_Straight_1x03
- removed P4: SATA_CON_L_13P, CenditFootprints2:SLIMLINE_SATA_PLUG_7P_6P
- removed P5: PORTCD_H_CON_7P, Pin_Headers:Pin_Header_Straight_1x07
- removed P6: PORTCD_L_CON_8P, Pin_Headers:Pin_Header_Straight_1x08
- removed P7: SATA_CON_R_13P, CenditFootprints:SATA_RECEPTACLE_VERTICAL_SMT_6P_7P
- removed the Q1 at (91.7, 120.2)
- removed the R1 at (261.4, 108.6)
- removed the R1 at (256.5, 48.9)
- removed the R1 at (33.0, 122.2)
- removed the R1 at (243.7, 134.5)
- removed the R1 at (177.8, 46.9)
- removed the R1 at (181.7, 182.5)
- removed the R10 at (253.2, 108.6)
- removed the R10 at (198.0, 40.6)
- removed the R10 at (173.4, 182.5)
- removed the R11 at (255.7, 87.8)
- removed the R11 at (197.9, 34.0)
- removed the R11 at (176.0, 161.6)
- removed the R12 at (261.0, 87.8)
- removed the R12 at (148.1, 63.4)
- removed the R12 at (181.3, 161.6)
- removed the R13 at (266.4, 87.8)
- removed the R13 at (145.9, 26.9)
- removed the R13 at (186.6, 161.6)
- removed the R14 at (271.6, 87.8)
- removed the R14 at (149.2, 26.9)
- removed the R14 at (191.9, 161.6)
- removed the R15 at (269.3, 108.6)
- removed the R15 at (182.6, 78.0)
- removed the R15 at (189.6, 182.5)
- removed the R16 at (264.0, 108.6)
- removed the R16 at (182.6, 80.8)
- removed the R16 at (184.2, 182.5)
- removed the R17 at (193.9, 61.7)
- removed the R17 at (136.7, 151.0)
- removed the R18 at (147.6, 31.6)
- removed the R18 at (152.9, 172.2)
- removed the R19 at (147.6, 34.2)
- removed the R19 at (150.6, 172.2)
- removed the R2 at (256.0, 108.6)
- removed the R2 at (62.9, 126.6)
- removed the R2 at (273.6, 138.9)
- removed the R2 at (177.8, 44.3)
- removed the R2 at (176.2, 182.5)
- removed the R20 at (147.6, 36.7)
- removed the R20 at (124.0, 183.3)
- removed the R21 at (147.6, 39.2)
- removed the R21 at (116.6, 156.8)
- removed the R22 at (147.6, 41.8)
- removed the R22 at (124.1, 118.5)
- removed the R23 at (147.6, 44.3)
- removed the R23 at (127.1, 118.5)
- removed the R24 at (183.5, 57.8)
- removed the R24 at (169.1, 136.4)
- removed the R25 at (180.5, 57.7)
- removed the R25 at (169.1, 125.1)
- removed the R26 at (186.3, 65.4)
- removed the R26 at (169.1, 131.1)
- removed the R27 at (163.3, 135.0)
- removed the R28 at (163.3, 132.5)
- removed the R29 at (206.0, 176.2)
- removed the R3 at (253.0, 87.8)
- removed the R3 at (39.4, 122.2)
- removed the R3 at (250.1, 134.5)
- removed the R3 at (177.8, 41.8)
- removed the R3 at (173.3, 161.6)
- removed the R30 at (166.1, 158.1)
- removed the R31 at (168.5, 155.6)
- removed the R32 at (91.8, 125.3)
- removed the R33 at (97.6, 119.3)
- removed the R4 at (258.4, 87.8)
- removed the R4 at (55.9, 154.6)
- removed the R4 at (266.6, 166.9)
- removed the R4 at (177.8, 39.2)
- removed the R4 at (178.6, 161.6)
- removed the R5 at (263.7, 87.8)
- removed the R5 at (39.4, 153.9)
- removed the R5 at (250.1, 166.2)
- removed the R5 at (177.8, 36.7)
- removed the R5 at (184.0, 161.6)
- removed the R6 at (268.9, 87.8)
- removed the R6 at (39.4, 160.3)
- removed the R6 at (250.1, 172.6)
- removed the R6 at (177.8, 34.2)
- removed the R6 at (189.2, 161.6)
- removed the R7 at (272.0, 108.6)
- removed the R7 at (177.8, 31.6)
- removed the R7 at (192.2, 182.5)
- removed the R8 at (266.6, 108.6)
- removed the R8 at (177.8, 29.1)
- removed the R8 at (186.9, 182.5)
- removed the R9 at (258.8, 108.6)
- removed the R9 at (198.0, 46.7)
- removed the R9 at (179.0, 182.5)
- removed the RS1 at (33.0, 128.5)
- removed the RS1 at (243.7, 140.8)
- removed the U1 at (262.8, 77.4)
- removed the U1 at (247.4, 40.4)
- removed the U1 at (40.6, 126.6)
- removed the U1 at (251.3, 138.9)
- removed the U1 at (154.7, 29.1)
- removed the U1 at (183.1, 151.2)
- removed the U2 at (48.3, 152.7)
- removed the U2 at (259.0, 165.0)
- removed the U2 at (141.5, 117.3)
- removed the U3 at (109.0, 178.7)
- removed U4: MC33996EKR2, CenditFootprints:MC33996-SOIC32
- removed U5: PCA6416A, CenditFootprints:PCA6416A-TSSOP24
- removed the Y1 at (143.4, 61.8)
- removed the Y1 at (132.0, 147.5)
- added C1: 0.1uF/10V, Capacitors_SMD:C_1206_HandSoldering, F.Cu at (157.9, 29.5)
- added C1: 0.1uF/30V, Capacitors_SMD:C_1206_HandSoldering, F.Cu at (31.6, 140.6)
- added C1: 0.1uF/30V, Capacitors_SMD:C_1206_HandSoldering, F.Cu at (31.0, 184.8)
- added C1: 100uF@50V, CenditFootprints2:C_Radial_D8_L13_P3.8, F.Cu at (98.2, 136.0)
- added C1: 100uF@50V, CenditFootprints2:C_Radial_D8_L13_P3.8, F.Cu at (156.0, 136.0)
- added C2: 0.1uF/10V, Capacitors_SMD:C_1206_HandSoldering, F.Cu at (165.9, 29.5)
- added C2: 0.1uF/10V, Capacitors_SMD:C_1206_HandSoldering, F.Cu at (27.9, 135.8)
- added C2: 0.1uF/10V, Capacitors_SMD:C_1206_HandSoldering, F.Cu at (27.3, 180.0)
- added C2: 100nF, Capacitors_SMD:C_0805_HandSoldering, F.Cu at (96.9, 143.0)
- added C2: 100nF, Capacitors_SMD:C_0805_HandSoldering, F.Cu at (154.7, 143.0)
- added C3: 0.3nF, Capacitors_SMD:C_0805_HandSoldering, F.Cu at (118.5, 124.0)
- added C3: 0.3nF, Capacitors_SMD:C_0805_HandSoldering, F.Cu at (176.3, 124.0)
- added C4: 470uF@10V, CenditFootprints2:C_Radial_D8_L13_P3.8, F.Cu at (126.1, 125.2)
- added C4: 470uF@10V, CenditFootprints2:C_Radial_D8_L13_P3.8, F.Cu at (183.9, 125.2)
- added C5: 100uF@10V, CenditFootprints2:C_Radial_D8_L13_P3.8, F.Cu at (128.7, 143.0)
- added C5: 100uF@10V, CenditFootprints2:C_Radial_D8_L13_P3.8, F.Cu at (186.4, 143.0)
- added C6: 100nF, Capacitors_SMD:C_0805_HandSoldering, F.Cu at (130.6, 150.0)
- added C6: 100nF, Capacitors_SMD:C_0805_HandSoldering, F.Cu at (188.3, 150.0)
- added C7: 100uF@10V, CenditFootprints2:C_Radial_D8_L13_P3.8, F.Cu at (102.6, 153.2)
- added C7: 100uF@10V, CenditFootprints2:C_Radial_D8_L13_P3.8, F.Cu at (160.4, 153.2)
- added C8: 100nF, Capacitors_SMD:C_0805_HandSoldering, F.Cu at (105.2, 160.1)
- added C8: 100nF, Capacitors_SMD:C_0805_HandSoldering, F.Cu at (162.9, 160.1)
- added C9: 1uF, Capacitors_SMD:C_0805_HandSoldering, F.Cu at (130.6, 154.4)
- added C9: 1uF, Capacitors_SMD:C_0805_HandSoldering, F.Cu at (188.3, 154.4)
- added D1: SPVH24, CenditFootprints:SPHV24-SOD882, F.Cu at (153.5, 49.7)
- added D1: DST5100S, CenditFootprints2:DST5100S-TO-277B, F.Cu at (104.5, 142.4)
- added D1: DST5100S, CenditFootprints2:DST5100S-TO-277B, F.Cu at (162.3, 142.4)
- added D10: SPVH24, CenditFootprints:SPHV24-SOD882, F.Cu at (159.1, 62.8)
- added D11: SPVH24, CenditFootprints:SPHV24-SOD882, F.Cu at (156.7, 62.8)
- added D12: SPVH24, CenditFootprints:SPHV24-SOD882, F.Cu at (153.7, 62.8)
- added D13: SPVH24, CenditFootprints:SPHV24-SOD882, F.Cu at (172.0, 62.8)
- added D14: SPVH24, CenditFootprints:SPHV24-SOD882, F.Cu at (169.4, 62.8)
- added D15: SPVH24, CenditFootprints:SPHV24-SOD882, F.Cu at (166.6, 62.8)
- added D16: SPVH24, CenditFootprints:SPHV24-SOD882, F.Cu at (164.1, 62.8)
- added D2: SPVH24, CenditFootprints:SPHV24-SOD882, F.Cu at (156.1, 49.6)
- added D2: SPHV24-01ETG, CenditFootprints2:SPHV24-SOD882, F.Cu at (99.6, 124.6)
- added D2: SPHV24-01ETG, CenditFootprints2:SPHV24-SOD882, F.Cu at (157.4, 124.6)
- added D3: SPVH24, CenditFootprints:SPHV24-SOD882, F.Cu at (158.7, 49.6)
- added D3: LED, LEDs:LED_0805, F.Cu at (134.4, 120.1)
- added D3: LED, LEDs:LED_0805, F.Cu at (192.2, 120.1)
- added D4: SPVH24, CenditFootprints:SPHV24-SOD882, F.Cu at (161.5, 49.6)
- added D5: SPVH24, CenditFootprints:SPHV24-SOD882, F.Cu at (164.1, 49.6)
- added D6: SPVH24, CenditFootprints:SPHV24-SOD882, F.Cu at (166.8, 49.6)
- added D7: SPVH24, CenditFootprints:SPHV24-SOD882, F.Cu at (169.4, 49.6)
- added D8: SPVH24, CenditFootprints:SPHV24-SOD882, F.Cu at (172.0, 49.6)
- added D9: SPVH24, CenditFootprints:SPHV24-SOD882, F.Cu at (161.6, 62.8)
- added J1: DEBUG_CON_01X08, CenditFootprints:DEBUG_CON_8P, F.Cu at (137.8, 37.3)
- added J1: DEBUG_CON_9P, CenditFootprints:DEBUG_CON_9P, F.Cu at (65.5, 124.0)
- added J1: DEBUG_CON_9P, CenditFootprints:DEBUG_CON_9P, F.Cu at (64.9, 168.1)
- added J2: GPIB_CON_9P, CenditFootprints:GPIB_HEADER_9P, F.Cu at (170.7, 54.5)
- added J2: VIKING_CON_9P, CenditFootprints:VIKING_HEADER_9P, F.Cu at (55.0, 125.6)
- added J2: VIKING_CON_9P, CenditFootprints:VIKING_HEADER_9P, F.Cu at (54.4, 169.8)
- added J3: GPIB_CON_9P, CenditFootprints:GPIB_HEADER_9P, F.Cu at (170.7, 57.9)
- added J3: VIKING_CON_9P, CenditFootprints:VIKING_HEADER_9P, F.Cu at (55.0, 122.2)
- added J3: VIKING_CON_9P, CenditFootprints:VIKING_HEADER_9P, F.Cu at (54.4, 166.4)
- added J4: SATA_CON_14P, CenditFootprints:SLIMLINE_SATA_PLUG_7P_6P, F.Cu at (73.3, 132.3)
- added J4: SATA_CON_14P, CenditFootprints:SLIMLINE_SATA_PLUG_7P_6P, F.Cu at (72.6, 176.5)
- added L1: 220uH, CenditFootprints2:INDUCTOR_LCM1060, F.Cu at (117.2, 137.9)
- added L1: 220uH, CenditFootprints2:INDUCTOR_LCM1060, F.Cu at (175.0, 137.9)
- added L2: 1uH, CenditFootprints2:INDUCTOR_LKS0745, F.Cu at (129.9, 133.5)
- added L2: 1uH, CenditFootprints2:INDUCTOR_LKS0745, F.Cu at (187.7, 133.5)
- added P1: PWR_IN_2P, Pin_Headers:Pin_Header_Straight_1x02, F.Cu at (96.3, 125.9)
- added P1: PWR_IN_2P, Pin_Headers:Pin_Header_Straight_1x02, F.Cu at (154.1, 125.9)
- added P2: PWR_OUT_4P, Pin_Headers:Pin_Header_Straight_1x04, F.Cu at (96.9, 153.2)
- added P2: PWR_OUT_4P, Pin_Headers:Pin_Header_Straight_1x04, F.Cu at (154.7, 153.2)
- added R1: 1k, Resistors_SMD:R_0805_HandSoldering, F.Cu at (160.8, 66.7)
- added R1: 1k, Resistors_SMD:R_0805_HandSoldering, F.Cu at (54.6, 145.2)
- added R1: 1k, Resistors_SMD:R_0805_HandSoldering, F.Cu at (54.0, 189.4)
- added R1: 2.0k, Resistors_SMD:R_0805_HandSoldering, F.Cu at (104.5, 122.0)
- added R1: 2.0k, Resistors_SMD:R_0805_HandSoldering, F.Cu at (162.3, 122.0)
- added R10: 1k, Resistors_SMD:R_0805_HandSoldering, F.Cu at (152.6, 66.7)
- added R11: 1k, Resistors_SMD:R_0805_HandSoldering, F.Cu at (155.1, 45.9)
- added R12: 1k, Resistors_SMD:R_0805_HandSoldering, F.Cu at (160.5, 45.9)
- added R13: 1k, Resistors_SMD:R_0805_HandSoldering, F.Cu at (165.8, 45.9)
- added R14: 1k, Resistors_SMD:R_0805_HandSoldering, F.Cu at (171.0, 45.9)
- added R15: 1k, Resistors_SMD:R_0805_HandSoldering, F.Cu at (168.7, 66.7)
- added R16: 1k, Resistors_SMD:R_0805_HandSoldering, F.Cu at (163.4, 66.7)
- added R2: 1k, Resistors_SMD:R_0805_HandSoldering, F.Cu at (155.4, 66.7)
- added R2: 330, Resistors_SMD:R_0805_HandSoldering, F.Cu at (134.4, 126.5)
- added R2: 330, Resistors_SMD:R_0805_HandSoldering, F.Cu at (192.2, 126.5)
- added R3: 1k, Resistors_SMD:R_0805_HandSoldering, F.Cu at (152.5, 45.9)
- added R3: 1.0k, Resistors_SMD:R_0805_HandSoldering, F.Cu at (110.9, 122.0)
- added R3: 1.0k, Resistors_SMD:R_0805_HandSoldering, F.Cu at (168.7, 122.0)
- added R4: 1k, Resistors_SMD:R_0805_HandSoldering, F.Cu at (157.8, 45.9)
- added R4: 10k, Resistors_SMD:R_0805_HandSoldering, F.Cu at (127.4, 154.4)
- added R4: 10k, Resistors_SMD:R_0805_HandSoldering, F.Cu at (185.2, 154.4)
- added R5: 1k, Resistors_SMD:R_0805_HandSoldering, F.Cu at (163.1, 45.9)
- added R5: 4.3k, Resistors_SMD:R_0805_HandSoldering, F.Cu at (110.9, 153.8)
- added R5: 4.3k, Resistors_SMD:R_0805_HandSoldering, F.Cu at (168.7, 153.8)
- added R6: 1k, Resistors_SMD:R_0805_HandSoldering, F.Cu at (168.3, 45.9)
- added R6: 3.0k, Resistors_SMD:R_0805_HandSoldering, F.Cu at (110.9, 160.1)
- added R6: 3.0k, Resistors_SMD:R_0805_HandSoldering, F.Cu at (168.7, 160.1)
- added R7: 1k, Resistors_SMD:R_0805_HandSoldering, F.Cu at (171.4, 66.7)
- added R8: 1k, Resistors_SMD:R_0805_HandSoldering, F.Cu at (166.1, 66.7)
- added R9: 1k, Resistors_SMD:R_0805_HandSoldering, F.Cu at (158.2, 66.7)
- added RS1: 0.20, Resistors_SMD:R_0805_HandSoldering, F.Cu at (104.5, 128.4)
- added RS1: 0.20, Resistors_SMD:R_0805_HandSoldering, F.Cu at (162.3, 128.4)
- added U1: PCA6416A, CenditFootprints:PCA6416A-TSSOP24, F.Cu at (162.2, 35.5)
- added U1: MC33996EKR2, CenditFootprints:MC33996-SOIC32, F.Cu at (45.5, 136.7)
- added U1: MC33996EKR2, CenditFootprints:MC33996-SOIC32, F.Cu at (44.8, 180.8)
- added U1: SP34063A, CenditFootprints2:SP34063AEN-L&slash_TR, F.Cu at (112.1, 126.5)
- added U1: SP34063A, CenditFootprints2:SP34063AEN-L&slash_TR, F.Cu at (169.9, 126.5)
- added U2: SPX29152, CenditFootprints2:SPX29152T5-TO-263-5, F.Cu at (119.8, 152.5)
- added U2: SPX29152, CenditFootprints2:SPX29152T5-TO-263-5, F.Cu at (177.5, 152.5)
- moved J4 109.0 mm to (131.6, 48.3)
- moved C3 2.54 mm to (81.0, 96.5)
- moved D4 2.54 mm to (94.8, 85.9)
- moved JP1 2.54 mm to (109.5, 87.4)
- moved R38 2.54 mm to (55.3, 80.7)
- moved R25 2.54 mm to (83.8, 51.7)
- moved R26 2.54 mm to (83.8, 49.1)
- moved R28 2.54 mm to (83.8, 44.1)
- moved BATT1 2.54 mm to (91.5, 22.5)
- moved C18 2.54 mm to (100.2, 22.5)
- moved C5 2.54 mm to (54.6, 29.0)
- moved CON2 2.54 mm to (73.3, 25.3)
- moved D6 2.54 mm to (111.1, 32.1)
- moved J1 2.54 mm to (50.9, 25.7)
- moved LS1 2.54 mm to (45.6, 28.1)
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Routing:
- net GND: track 1839.3 -> 545.5 mm, vias 72 -> 23
- net VDD: track 1128.2 -> 525.0 mm, vias 30 -> 13
- net GNDPWR: track 1476.4 -> 1308.9 mm, vias 16 -> 12
- net +24.0V: track 332.9 -> 223.6 mm, vias 16 -> 10
- net /SPI_SCLK: track 107.8 -> 0.00 mm, vias 4 -> 0
- net //INT: track 144.3 -> 45.4 mm, vias 5 -> 2
- net /SCL: track 174.1 -> 75.6 mm
- net /SDA: track 165.9 -> 68.9 mm, vias 4 -> 2
- net VBUS: track 76.4 -> 0.00 mm, vias 2 -> 0
- net /U4_CS: track 72.1 -> 0.00 mm, vias 2 -> 0
- net /U3_CS: track 69.0 -> 0.00 mm, vias 2 -> 0
- net /PD3: track 59.9 -> 0.00 mm, vias 2 -> 0
- net /MOSI: track 159.0 -> 100.6 mm, vias 6 -> 4
- net Net-(R16-Pad2): track 110.4 -> 55.2 mm
- net /VKY7: track 55.1 -> 0.00 mm
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Other:
- net class GND removed
- net class IOPORT removed
- net class POWER removed
- net class PWR added: clearance 0.3, trace_width 1, via_dia 1.6, via_drill 0.4
- net class SIGNAL added: clearance 0.3, trace_width 0.5, via_dia 1.6, via_drill 0.4
- net class VIKING removed
- rule pad_to_mask_clearance: 0.2 -> 0
- board text added: "CAPA BOTTOM INVERTIR DERECHA CON IZQUIERDA"
- board text added: "CAPA TOP NO INVERTIR"
- board text added: "CENDIT"
- board text added: "CORREO@JOSEARIAS.COM.VE"

Commit message: Revision de PCBs + generacion nuevos gerber
  - Se hacen ligeras correcciones en los PCBs (5)
  - Se genera nuevamente archivo PCBs combinados
  - Se generan nuevos archivos gerber
Parts:
- removed the C1 at (31.6, 140.6)
- removed the C1 at (31.0, 184.8)
- removed the C1 at (98.2, 136.0)
- removed the C1 at (156.0, 136.0)
- removed the C2 at (27.9, 135.8)
- removed the C2 at (27.3, 180.0)
- removed the C2 at (96.9, 143.0)
- removed the C2 at (154.7, 143.0)
- removed the C3 at (118.5, 124.0)
- removed the C3 at (176.3, 124.0)
- removed the C4 at (126.1, 125.2)
- removed the C4 at (183.9, 125.2)
- removed the C5 at (128.7, 143.0)
- removed the C5 at (186.4, 143.0)
- removed the C6 at (130.6, 150.0)
- removed the C6 at (188.3, 150.0)
- removed the C7 at (102.6, 153.2)
- removed the C7 at (160.4, 153.2)
- removed the C8 at (105.2, 160.1)
- removed the C8 at (162.9, 160.1)
- removed the C9 at (130.6, 154.4)
- removed the C9 at (188.3, 154.4)
- removed the D1 at (104.5, 142.4)
- removed the D1 at (162.3, 142.4)
- removed the D2 at (99.6, 124.6)
- removed the D2 at (157.4, 124.6)
- removed the D3 at (134.4, 120.1)
- removed the D3 at (192.2, 120.1)
- removed the J1 at (65.5, 124.0)
- removed the J1 at (64.9, 168.1)
- removed the J2 at (55.0, 125.6)
- removed the J2 at (54.4, 169.8)
- removed the J3 at (55.0, 122.2)
- removed the J3 at (54.4, 166.4)
- removed the J4 at (73.3, 132.3)
- removed the J4 at (72.6, 176.5)
- removed the L1 at (117.2, 137.9)
- removed the L1 at (175.0, 137.9)
- removed the L2 at (129.9, 133.5)
- removed the L2 at (187.7, 133.5)
- removed the P1 at (96.3, 125.9)
- removed the P1 at (154.1, 125.9)
- removed the P2 at (96.9, 153.2)
- removed the P2 at (154.7, 153.2)
- removed the R1 at (54.6, 145.2)
- removed the R1 at (54.0, 189.4)
- removed the R1 at (104.5, 122.0)
- removed the R1 at (162.3, 122.0)
- removed the R2 at (134.4, 126.5)
- removed the R2 at (192.2, 126.5)
- removed the R3 at (110.9, 122.0)
- removed the R3 at (168.7, 122.0)
- removed the R4 at (127.4, 154.4)
- removed the R4 at (185.2, 154.4)
- removed the R5 at (110.9, 153.8)
- removed the R5 at (168.7, 153.8)
- removed the R6 at (110.9, 160.1)
- removed the R6 at (168.7, 160.1)
- removed the RS1 at (104.5, 128.4)
- removed the RS1 at (162.3, 128.4)
- removed the U1 at (45.5, 136.7)
- removed the U1 at (44.8, 180.8)
- removed the U1 at (112.1, 126.5)
- removed the U1 at (169.9, 126.5)
- removed the U2 at (119.8, 152.5)
- removed the U2 at (177.5, 152.5)
- added C1: 0.1uF/30V, Capacitors_SMD:C_1206_HandSoldering, F.Cu at (143.8, 50.9)
- added C1: 0.1uF/30V, Capacitors_SMD:C_1206_HandSoldering, F.Cu at (143.5, 95.6)
- added C1: 100uF@50V, CenditFootprints2:C_Radial_D8_L13_P3.8, F.Cu at (93.3, 140.2)
- added C1: 100uF@50V, CenditFootprints2:C_Radial_D8_L13_P3.8, F.Cu at (153.3, 139.4)
- added C2: 0.1uF/10V, Capacitors_SMD:C_1206_HandSoldering, F.Cu at (140.1, 46.1)
- added C2: 0.1uF/10V, Capacitors_SMD:C_1206_HandSoldering, F.Cu at (139.8, 90.8)
- added C2: 100nF, Capacitors_SMD:C_0805_HandSoldering, F.Cu at (92.1, 147.2)
- added C2: 100nF, Capacitors_SMD:C_0805_HandSoldering, F.Cu at (152.0, 146.4)
- added C3: 0.3nF, Capacitors_SMD:C_0805_HandSoldering, F.Cu at (113.7, 128.1)
- added C3: 0.3nF, Capacitors_SMD:C_0805_HandSoldering, F.Cu at (173.6, 127.4)
- added C4: 470uF@10V, CenditFootprints2:C_Radial_D8_L13_P3.8, F.Cu at (121.3, 129.4)
- added C4: 470uF@10V, CenditFootprints2:C_Radial_D8_L13_P3.8, F.Cu at (181.2, 128.7)
- added C5: 100uF@10V, CenditFootprints2:C_Radial_D8_L13_P3.8, F.Cu at (123.8, 147.2)
- added C5: 100uF@10V, CenditFootprints2:C_Radial_D8_L13_P3.8, F.Cu at (183.8, 146.4)
- added C6: 100nF, Capacitors_SMD:C_0805_HandSoldering, F.Cu at (125.7, 154.2)
- added C6: 100nF, Capacitors_SMD:C_0805_HandSoldering, F.Cu at (185.7, 153.4)
- added C7: 100uF@10V, CenditFootprints2:C_Radial_D8_L13_P3.8, F.Cu at (97.8, 157.4)
- added C7: 100uF@10V, CenditFootprints2:C_Radial_D8_L13_P3.8, F.Cu at (157.7, 156.6)
- added C8: 100nF, Capacitors_SMD:C_0805_HandSoldering, F.Cu at (100.3, 164.3)
- added C8: 100nF, Capacitors_SMD:C_0805_HandSoldering, F.Cu at (160.3, 163.6)
- added C9: 1uF, Capacitors_SMD:C_0805_HandSoldering, F.Cu at (127.5, 160.0)
- added C9: 1uF, Capacitors_SMD:C_0805_HandSoldering, F.Cu at (187.5, 159.3)
- added D1: DST5100S, CenditFootprints2:DST5100S-TO-277B, F.Cu at (99.7, 146.6)
- added D1: DST5100S, CenditFootprints2:DST5100S-TO-277B, F.Cu at (159.6, 145.8)
- added D2: SPHV24-01ETG, CenditFootprints2:SPHV24-SOD882, F.Cu at (94.7, 128.8)
- added D2: SPHV24-01ETG, CenditFootprints2:SPHV24-SOD882, F.Cu at (154.7, 128.0)
- added D3: LED, LEDs:LED_0805, F.Cu at (129.5, 124.3)
- added D3: LED, LEDs:LED_0805, F.Cu at (189.5, 123.6)
- added J1: DEBUG_CON_9P, CenditFootprints:DEBUG_CON_9P, F.Cu at (177.7, 34.3)
- added J1: DEBUG_CON_9P, CenditFootprints:DEBUG_CON_9P, F.Cu at (177.4, 79.0)
- added J2: VIKING_CON_9P, CenditFootprints:VIKING_HEADER_9P, F.Cu at (167.1, 35.9)
- added J2: VIKING_CON_9P, CenditFootprints:VIKING_HEADER_9P, F.Cu at (166.9, 80.6)
- added J3: VIKING_CON_9P, CenditFootprints:VIKING_HEADER_9P, F.Cu at (167.1, 32.5)
- added J3: VIKING_CON_9P, CenditFootprints:VIKING_HEADER_9P, F.Cu at (166.9, 77.2)
- added J4: SATA_CON_14P, CenditFootprints:SLIMLINE_SATA_PLUG_7P_6P, F.Cu at (185.4, 42.7)
- added J4: SATA_CON_14P, CenditFootprints:SLIMLINE_SATA_PLUG_7P_6P, F.Cu at (185.2, 87.4)
- added L1: 220uH, CenditFootprints2:INDUCTOR_LCM1060, F.Cu at (112.4, 142.1)
- added L1: 220uH, CenditFootprints2:INDUCTOR_LCM1060, F.Cu at (172.3, 141.4)
- added L2: 1uH, CenditFootprints2:INDUCTOR_LKS0745, F.Cu at (125.1, 137.7)
- added L2: 1uH, CenditFootprints2:INDUCTOR_LKS0745, F.Cu at (185.0, 136.9)
- added P1: PWR_IN_2P, Pin_Headers:Pin_Header_Straight_1x02, F.Cu at (91.4, 130.0)
- added P1: PWR_IN_2P, Pin_Headers:Pin_Header_Straight_1x02, F.Cu at (151.4, 129.3)
- added P2: PWR_OUT_4P, Pin_Headers:Pin_Header_Straight_1x04, F.Cu at (92.1, 157.4)
- added P2: PWR_OUT_4P, Pin_Headers:Pin_Header_Straight_1x04, F.Cu at (152.0, 156.6)
- added R1: 1k, Resistors_SMD:R_0805_HandSoldering, F.Cu at (166.8, 55.5)
- added R1: 1k, Resistors_SMD:R_0805_HandSoldering, F.Cu at (166.5, 100.2)
- added R1: 2.0k, Resistors_SMD:R_0805_HandSoldering, F.Cu at (99.7, 126.2)
- added R1: 2.0k, Resistors_SMD:R_0805_HandSoldering, F.Cu at (159.6, 125.5)
- added R2: 330, Resistors_SMD:R_0805_HandSoldering, F.Cu at (129.5, 130.7)
- added R2: 330, Resistors_SMD:R_0805_HandSoldering, F.Cu at (189.5, 129.9)
- added R3: 1.0k, Resistors_SMD:R_0805_HandSoldering, F.Cu at (106.0, 126.2)
- added R3: 1.0k, Resistors_SMD:R_0805_HandSoldering, F.Cu at (166.0, 125.5)
- added R4: 10k, Resistors_SMD:R_0805_HandSoldering, F.Cu at (124.5, 160.0)
- added R4: 10k, Resistors_SMD:R_0805_HandSoldering, F.Cu at (184.4, 159.3)
- added R5: 4.3k, Resistors_SMD:R_0805_HandSoldering, F.Cu at (106.0, 158.0)
- added R5: 4.3k, Resistors_SMD:R_0805_HandSoldering, F.Cu at (166.0, 157.2)
- added R6: 3.0k, Resistors_SMD:R_0805_HandSoldering, F.Cu at (106.0, 164.3)
- added R6: 3.0k, Resistors_SMD:R_0805_HandSoldering, F.Cu at (166.0, 163.6)
- added RS1: 0.20, Resistors_SMD:R_0805_HandSoldering, F.Cu at (99.7, 132.6)
- added RS1: 0.20, Resistors_SMD:R_0805_HandSoldering, F.Cu at (159.6, 131.8)
- added U1: MC33996EKR2, CenditFootprints:MC33996-SOIC32, F.Cu at (157.6, 47.0)
- added U1: MC33996EKR2, CenditFootprints:MC33996-SOIC32, F.Cu at (157.4, 91.7)
- added U1: SP34063A, CenditFootprints2:SP34063AEN-L&slash_TR, F.Cu at (107.3, 130.7)
- added U1: SP34063A, CenditFootprints2:SP34063AEN-L&slash_TR, F.Cu at (167.3, 129.9)
- added U2: SPX29152, CenditFootprints2:SPX29152T5-TO-263-5, F.Cu at (114.9, 156.7)
- added U2: SPX29152, CenditFootprints2:SPX29152T5-TO-263-5, F.Cu at (174.9, 156.0)
- moved D1 142.0 mm to (50.9, 147.9)
- moved D13 142.0 mm to (69.4, 161.0)
- moved D14 142.0 mm to (66.7, 161.0)
- moved D2 142.0 mm to (53.5, 147.8)
- moved D7 142.0 mm to (66.7, 147.8)
- moved D8 142.0 mm to (69.4, 147.8)
- moved J4 142.0 mm to (29.0, 146.4)
- moved R11 142.0 mm to (52.5, 144.1)
- moved R14 142.0 mm to (68.4, 144.1)
- moved R15 142.0 mm to (66.1, 164.9)
- moved R16 142.0 mm to (60.8, 164.9)
- moved R2 142.0 mm to (52.8, 164.9)
- moved R3 142.0 mm to (49.8, 144.1)
- moved R4 142.0 mm to (55.2, 144.1)
- moved R6 142.0 mm to (65.7, 144.1)
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Connections:
- R30 pad 2: /PB5 -> GNDD
Routing:
- net /ENABLE: track 132.9 -> 152.4 mm
- net GNDD: track 859.5 -> 871.1 mm, vias 18 -> 19
- net Net-(C4-Pad1): track 92.7 -> 82.8 mm
- net Net-(D1-Pad1): track 52.5 -> 60.2 mm
- net GNDPWR: track 1308.9 -> 1302.6 mm
- net /PB6: track 32.5 -> 31.2 mm
- net VREG: track 195.2 -> 195.8 mm
